Commit message: feat: Arduino homing sequence – edge-approach algorithm, robust protocol & zeroing
Reworks the axis-1 homing into a reliable, encoder-agnostic sequence.

Arduino firmware (r0192_homing.ino):
- Single axis-specific CAN ID for RX+TX; meaning in Data[0]
  (CMD_ARM 0x01 / RSP_DETECTED 0xFF / RSP_ERROR 0xEE)
- Timeout so the node never hangs when no magnet is seen
- Debug logging filtered to the node's own CAN ID

Homing (extracted into HomingController, own node + executor):
- Two-sided edge approach: edge A -> overshoot -> edge B -> midpoint
- Ramped position setpoints for sweep and moves (search_kp / move_vel)
  so the motor drives itself slowly instead of stalling or snapping
- Pre-check "already on magnet" -> back off before Pass 1
- Range check at start (max_start_angle, ±180°) + configurable search_dir
  to keep the magnet unique despite the continuous multi-turn encoder
- arm_controller deactivated/reactivated via switch_controller so it does
  not fight homing or snap back to the stale pre-homing setpoint
- Whole arm set to the home pose (all joints 0) after homing

GDS68 driver:
- Software home offset (set_home_offset/set_home_here); get_current_position
  reports raw-offset, MIT_Control adds it back. Set_Linear_Count(0) does not
  persist on the absolute/continuous encoder.

URDF:
- joint_1 axis flipped to 0 0 -1 so the RViz model turns with the real motor.

CLAUDE.md updated throughout (protocol, algorithm, params, gotchas, tasks).

Co-Authored-By: Claude Opus 4.8 <noreply@anthropic.com>

File: src/r0192_description/urdf/r0192.urdf.xacro (robot description, xacro)
@@ -200,5 +200,7 @@
         <child link="link_1" />
         <origin xyz="0 0 1.751" />
-        <axis xyz="0 0 1" />
+        <!-- -Z: motor's positive rotation is opposite the model's default +Z,
+             so the RViz model turns the same way as the physical axis 1. -->
+        <axis xyz="0 0 -1" />
         <limit lower="-${PI}" upper="${PI}"
             effort="${effort}" velocity="${velocity}" />
