Commit message: Refactor RS05Driver and GDS68Driver integration, enhance CAN communication handling, and update MoveIt configuration
- Implemented placeholder return values for unimplemented functions in RS05Driver.
- Added thread safety for feedback frame processing in RS05Driver.
- Updated CMakeLists.txt to remove unnecessary dependencies and streamline build process.
- Increased update rate in r0192_controllers.yaml for improved control responsiveness.
- Adjusted joint limits in URDF files for gripper joints to ensure correct operation.
- Enhanced r0192_ros2_control.xacro for better simulation and real robot handling.
- Created r0192_hardware package with a shared library for hardware interface.
- Implemented joint index mapping for efficient access in R0192SystemHardware.
- Improved read/write methods in R0192SystemHardware for better handling of joint states.
- Added CAN communication availability checks and logging for better diagnostics.
- Updated MoveIt configuration files for improved planning and execution.
- Introduced a new hardware plugin XML file for r0192_hardware.

File: src/r0192_description/urdf/r0192.urdf.xacro (robot description, xacro)
@@ -255,5 +255,5 @@
         <origin xyz="0 0 0"/>
         <axis xyz="0 1 0"/>
-        <limit lower="0.15" upper="0.0"
+        <limit lower="0.0" upper="0.025"
                effort="${effort}" velocity="${velocity}"/>
     </joint>
@@ -263,5 +263,5 @@
         <origin xyz="0 0 0"/>
         <axis xyz="0 1 0"/>
-        <limit lower="0.0" upper="-0.15"
+        <limit lower="-0.025" upper="0.0"
                effort="${effort}" velocity="${velocity}"/>
         <mimic joint="joint_7" multiplier="-1"/>

File: src/r0192_description/urdf/r0192_ros2_control.xacro (robot description, xacro)
@@ -1,10 +1,7 @@
 <?xml version="1.0"?>
 <robot xmlns:xacro="http://www.ros.org/wiki/xacro" name="r0192">
-<!-- Noch bei Bedarf für Simulation anpassen -->
     <ros2_control name="RobotSystem" type="system">
-        <xacro:property name="PI" value="3.14159265359" />
-        <!-- ros2_control Gazebo -->
+        <!-- Simulation (Gazebo Iron / ROS 2 Iron+) -->
         <xacro:if value="$(arg is_sim)">
-            <!-- ROS 2 Iron or above -->
             <xacro:unless value="$(arg is_ignition)">
                 <hardware>
@@ -12,43 +9,71 @@
                 </hardware>
             </xacro:unless>
-            <joint name="joint_5">
-                <param name="mimic">joint_4</param>
+            <!-- Gripper mimic for simulation -->
+            <joint name="joint_8">
+                <param name="mimic">joint_7</param>
                 <param name="multiplier">-1</param>
+                <command_interface name="position"/>
+                <state_interface name="position"/>
             </joint>
         </xacro:if>
-        <!-- ros2_control Real Robot -->
+        <!-- Real robot: r0192_hardware plugin via SocketCAN -->
         <xacro:unless value="$(arg is_sim)">
             <hardware>
-                <plugin>r0192_controller/r0192Interface</plugin>
-                <param name="port">/dev/ttyACM0</param>
+                <plugin>r0192_hardware/R0192SystemHardware</plugin>
             </hardware>
+            <!-- joint_8: passive mimic of joint_7, state only -->
+            <joint name="joint_8">
+                <state_interface name="position"/>
+                <state_interface name="velocity"/>
+            </joint>
         </xacro:unless>
+        <!-- Arm joints 1-6 (same for sim and real) -->
         <joint name="joint_1">
-            <command_interface name="position">
-            <param name="min">-${PI / 2}</param>
-            <param name="max">${PI / 2}</param>
-            </command_interface>
+            <command_interface name="position"/>
+            <command_interface name="velocity"/>
             <state_interface name="position"/>
+            <state_interface name="velocity"/>
+            <state_interface name="effort"/>
         </joint>
         <joint name="joint_2">
-            <command_interface name="position">
-            <param name="min">-${PI / 2}</param>
-            <param name="max">${PI / 2}</param>
-            </command_interface>
+            <command_interface name="position"/>
+            <command_interface name="velocity"/>
             <state_interface name="position"/>
+            <state_interface name="velocity"/>
+            <state_interface name="effort"/>
         </joint>
         <joint name="joint_3">
-            <command_interface name="position">
-            <param name="min">-${PI / 2}</param>
-            <param name="max">${PI / 2}</param>
-            </command_interface>
+            <command_interface name="position"/>
+            <command_interface name="velocity"/>
             <state_interface name="position"/>
+            <state_interface name="velocity"/>
+            <state_interface name="effort"/>
         </joint>
         <joint name="joint_4">
-            <command_interface name="position">
-            <param name="min">-${PI / 2}</param>
-            <param name="max">0.0</param>
-            </command_interface>
+            <command_interface name="position"/>
+            <command_interface name="velocity"/>
             <state_interface name="position"/>
+            <state_interface name="velocity"/>
+            <state_interface name="effort"/>
+        </joint>
+        <joint name="joint_5">
+            <command_interface name="position"/>
+            <command_interface name="velocity"/>
+            <state_interface name="position"/>
+            <state_interface name="velocity"/>
+            <state_interface name="effort"/>
+        </joint>
+        <joint name="joint_6">
+            <command_interface name="position"/>
+            <command_interface name="velocity"/>
+            <state_interface name="position"/>
+            <state_interface name="velocity"/>
+            <state_interface name="effort"/>
+        </joint>
+        <!-- Gripper (joint_7 active, joint_8 passive mimic defined above) -->
+        <joint name="joint_7">
+            <command_interface name="position"/>
+            <state_interface name="position"/>
+            <state_interface name="velocity"/>
         </joint>
     </ros2_control>

Commit message: Add JogPanel for teach-pendant style jogging and integrate MoveIt Servo
- Introduced a new JogPanel in r0192_rviz_plugins for controlling the R0192 arm via teach-pendant style jogging.
- Implemented joint and Cartesian jogging modes with corresponding buttons and a speed slider.
- Integrated the JogPanel with MoveIt Servo for real-time control, allowing for smooth operation while maintaining safety.
- Updated launch files to include the new servo_node for handling jogging commands.
- Modified URDF to add a TCP link for tool frame reference.
- Enhanced the r0192_hardware_interface to ensure motors remain disabled after activation until explicitly enabled by the operator.
- Adjusted RViz configuration to accommodate the new JogPanel and improved visualization settings.
- Added servo configuration file to manage command timing, scaling, and collision checking.

File: src/r0192_description/urdf/r0192.urdf.xacro (robot description, xacro)
@@ -269,3 +269,16 @@
         <mimic joint="joint_7" multiplier="-1"/>
     </joint>
+    <!-- TCP / tool frame (ROS-Industrial tool0 convention): +Z points along the
+         gripper approach (thrust) direction so Tool-mode jogging treats +Z as
+         approach, +Y as the finger open/close axis. gripper_base's own X is the
+         approach axis, so rotate +90° about Y to map the new Z onto X. Pure TF
+         frame (no visual/collision); not part of the r0192_arm IK chain, used
+         by MoveIt Servo as the Tool jog frame. Position sits at gripper_base;
+         move it to the real fingertip TCP once CAD values are available. -->
+    <link name="tcp"/>
+    <joint name="gripper_base_to_tcp" type="fixed">
+        <parent link="gripper_base"/>
+        <child link="tcp"/>
+        <origin xyz="0 0 0" rpy="0 ${PI / 2} 0"/>
+    </joint>
 </robot>

Commit message: Refactor URDF and RViz configurations for real-scale implementation
- Updated joint limits for joint_7 in CLAUDE.md and URDF to reflect real dimensions (0.0025 m).
- Adjusted URDF geometry scaling to 1:1 with real measurements, modifying mesh scales and joint origins accordingly.
- Revised MoveIt configuration to restore default singularity thresholds, now suitable for real-scale links.
- Enhanced RViz configuration for improved visualization, including adjustments to grid size and view settings.
- Implemented live readout for joint angles and TCP pose in jog_panel, utilizing TF for real-time updates.
- Added necessary dependencies for sensor_msgs and tf2 in CMakeLists.txt and package.xml.

File: src/r0192_description/urdf/r0192.urdf.xacro (robot description, xacro)
@@ -13,4 +13,7 @@
     <xacro:property name="effort" value="30.0" />        <!-- später noch mit echten Werten anpassen! -->
     <xacro:property name="velocity" value="10.0" />      <!-- später noch mit echten Werten anpassen! -->
+    <!-- STL meshes are exported in mm → 0.001 maps them to metres (1:1 real
+         size). Joint origins below are likewise in metres at real scale. -->
+    <xacro:property name="mesh_scale" value="0.001 0.001 0.001" />
     <!-- Useful Macros -->
     <xacro:macro name="default_inertial" params="mass">
@@ -31,5 +34,5 @@
             <geometry>
                 <mesh filename="package://r0192_description/meshes/visual/axis_1.stl"
-                    scale="0.01 0.01 0.01" />
+                    scale="${mesh_scale}" />
             </geometry>
         </visual>
@@ -38,5 +41,5 @@
             <geometry>
                 <mesh filename="package://r0192_description/meshes/collision/axis_1_collision.stl"
-                    scale="0.01 0.01 0.01" />
+                    scale="${mesh_scale}" />
             </geometry>
         </collision>
@@ -48,5 +51,5 @@
             <geometry>
                 <mesh filename="package://r0192_description/meshes/visual/axis_2.stl"
-                    scale="0.01 0.01 0.01" />
+                    scale="${mesh_scale}" />
             </geometry>
         </visual>
@@ -55,5 +58,5 @@
             <geometry>
                 <mesh filename="package://r0192_description/meshes/collision/axis_2_collision.stl"
-                    scale="0.01 0.01 0.01" />
+                    scale="${mesh_scale}" />
             </geometry>
         </collision>
@@ -65,5 +68,5 @@
             <geometry>
                 <mesh filename="package://r0192_description/meshes/visual/axis_3.stl"
-                    scale="0.01 0.01 0.01" />
+                    scale="${mesh_scale}" />
             </geometry>
         </visual>
@@ -72,5 +75,5 @@
             <geometry>
                 <mesh filename="package://r0192_description/meshes/collision/axis_3_collision.stl"
-                    scale="0.01 0.01 0.01" />
+                    scale="${mesh_scale}" />
             </geometry>
         </collision>
@@ -82,5 +85,5 @@
             <geometry>
                 <mesh filename="package://r0192_description/meshes/visual/axis_4.stl"
-                    scale="0.01 0.01 0.01" />
+                    scale="${mesh_scale}" />
             </geometry>
         </visual>
@@ -89,5 +92,5 @@
             <geometry>
                 <mesh filename="package://r0192_description/meshes/collision/axis_4_collision.stl"
-                    scale="0.01 0.01 0.01" />
+                    scale="${mesh_scale}" />
             </geometry>
         </collision>
@@ -99,5 +102,5 @@
             <geometry>
                 <mesh filename="package://r0192_description/meshes/visual/axis_5.stl"
-                    scale="0.01 0.01 0.01" />
+                    scale="${mesh_scale}" />
             </geometry>
         </visual>
@@ -106,5 +109,5 @@
             <geometry>
                 <mesh filename="package://r0192_description/meshes/collision/axis_5_collision.stl"
-                    scale="0.01 0.01 0.01" />
+                    scale="${mesh_scale}" />
             </geometry>
         </collision>
@@ -116,5 +119,5 @@
             <geometry>
                 <mesh filename="package://r0192_description/meshes/visual/axis_6.stl"
-                    scale="0.01 0.01 0.01" />
+                    scale="${mesh_scale}" />
             </geometry>
         </visual>
@@ -123,5 +126,5 @@
             <geometry>
                 <mesh filename="package://r0192_description/meshes/collision/axis_6_collision.stl"
-                    scale="0.01 0.01 0.01" />
+                    scale="${mesh_scale}" />
             </geometry>
         </collision>
@@ -133,5 +136,5 @@
             <geometry>
                 <mesh filename="package://r0192_description/meshes/visual/flansch.stl"
-                    scale="0.01 0.01 0.01" />
+                    scale="${mesh_scale}" />
             </geometry>
         </visual>
@@ -140,5 +143,5 @@
             <geometry>
                 <mesh filename="package://r0192_description/meshes/collision/flansch_collision.stl"
-                    scale="0.01 0.01 0.01" />
+                    scale="${mesh_scale}" />
             </geometry>
         </collision>
@@ -150,11 +153,11 @@
             <origin rpy="0 ${PI} ${PI / 2}" xyz="0 0 0"/>
             <geometry>
-                <mesh filename="package://r0192_description/meshes/gripper/gripper_base.stl" scale="0.01 0.01 0.01"/>
-            </geometry>
-        </visual>
-        <collision>
-            <origin rpy="0 ${PI} ${PI / 2}" xyz="0 0 0"/>
-            <geometry>
-                <mesh filename="package://r0192_description/meshes/gripper/gripper_base.stl" scale="0.01 0.01 0.01"/>
+                <mesh filename="package://r0192_description/meshes/gripper/gripper_base.stl" scale="${mesh_scale}"/>
+            </geometry>
+        </visual>
+        <collision>
+            <origin rpy="0 ${PI} ${PI / 2}" xyz="0 0 0"/>
+            <geometry>
+                <mesh filename="package://r0192_description/meshes/gripper/gripper_base.stl" scale="${mesh_scale}"/>
             </geometry>
         </collision>
@@ -165,11 +168,11 @@
             <origin rpy="0 ${PI} ${PI / 2}" xyz="0 0 0"/>
             <geometry>
-                <mesh filename="package://r0192_description/meshes/gripper/gripper_right.stl" scale="0.01 0.01 0.01"/>
-            </geometry>
-        </visual>
-        <collision>
-            <origin rpy="0 ${PI} ${PI / 2}" xyz="0 0 0"/>
-            <geometry>
-                <mesh filename="package://r0192_description/meshes/gripper/gripper_right.stl" scale="0.01 0.01 0.01"/>
+                <mesh filename="package://r0192_description/meshes/gripper/gripper_right.stl" scale="${mesh_scale}"/>
+            </geometry>
+        </visual>
+        <collision>
+            <origin rpy="0 ${PI} ${PI / 2}" xyz="0 0 0"/>
+            <geometry>
+                <mesh filename="package://r0192_description/meshes/gripper/gripper_right.stl" scale="${mesh_scale}"/>
             </geometry>
         </collision>
@@ -180,11 +183,11 @@
             <origin rpy="0 ${PI} ${PI / 2}" xyz="0 0 0"/>
             <geometry>
-                <mesh filename="package://r0192_description/meshes/gripper/gripper_left.stl" scale="0.01 0.01 0.01"/>
-            </geometry>
-        </visual>
-        <collision>
-            <origin rpy="0 ${PI} ${PI / 2}" xyz="0 0 0"/>
-            <geometry>
-                <mesh filename="package://r0192_description/meshes/gripper/gripper_left.stl" scale="0.01 0.01 0.01"/>
+                <mesh filename="package://r0192_description/meshes/gripper/gripper_left.stl" scale="${mesh_scale}"/>
+            </geometry>
+        </visual>
+        <collision>
+            <origin rpy="0 ${PI} ${PI / 2}" xyz="0 0 0"/>
+            <geometry>
+                <mesh filename="package://r0192_description/meshes/gripper/gripper_left.stl" scale="${mesh_scale}"/>
             </geometry>
         </collision>
@@ -199,5 +202,5 @@
         <parent link="base_link" />
         <child link="link_1" />
-        <origin xyz="0 0 1.751" />
+        <origin xyz="0 0 0.1751" />
         <!-- -Z: motor's positive rotation is opposite the model's default +Z,
              so the RViz model turns the same way as the physical axis 1. -->
@@ -209,5 +212,5 @@
         <parent link="link_1" />
         <child link="link_2" />
-        <origin xyz="0 1.4 0" />
+        <origin xyz="0 0.14 0" />
         <axis xyz="0 1 0" />
         <limit lower="-${PI / 2}" upper="${PI / 2}"
@@ -217,5 +220,5 @@
         <parent link="link_2" />
         <child link="link_3" />
-        <origin xyz="0 -1.252 1.85" />
+        <origin xyz="0 -0.1252 0.185" />
         <axis xyz="0 1 0" />
         <limit lower="-${PI / 4}" upper="${5 * PI / 4}"
@@ -225,5 +228,5 @@
         <parent link="link_3" />
         <child link="link_4" />
-        <origin xyz="-1.25 0 0" />
+        <origin xyz="-0.125 0 0" />
         <axis xyz="1 0 0" />
         <limit lower="-${PI}" upper="${PI}"
@@ -233,5 +236,5 @@
         <parent link="link_4" />
         <child link="link_5" />
-        <origin xyz="-1.4 0 0" />
+        <origin xyz="-0.14 0 0" />
         <axis xyz="0 1 0" />
         <limit lower="-${PI}" upper="${PI}"
@@ -250,5 +253,5 @@
         <parent link="link_6"/>
         <child link = "gripper_base"/>
-        <origin xyz="-1.19143 0 0.12234"/>
+        <origin xyz="-0.119143 0 0.012234"/>
     </joint>
     <joint name ="joint_7" type="prismatic">
@@ -257,5 +260,5 @@
         <origin xyz="0 0 0"/>
         <axis xyz="0 1 0"/>
-        <limit lower="0.0" upper="0.025"
+        <limit lower="0.0" upper="0.0025"
                effort="${effort}" velocity="${velocity}"/>
     </joint>
@@ -265,5 +268,5 @@
         <origin xyz="0 0 0"/>
         <axis xyz="0 1 0"/>
-        <limit lower="-0.025" upper="0.0"
+        <limit lower="-0.0025" upper="0.0"
                effort="${effort}" velocity="${velocity}"/>
         <mimic joint="joint_7" multiplier="-1"/>
