File: PCB/KiCad/_restore_backup_2026-09-08T17-39-47-741/DriverDasyChain.kicad_sch (KiCad schematic)
At the start: 44 parts, among them J1 Conn_01x03, J10 Conn_01x04, J12 Conn_01x04, J2 Conn_01x03, J3 Conn_01x03, J4 Conn_01x04, J5 Conn_01x03, J6 Conn_01x04, Q2 Q_NMOS_GDS, SW1 SW_DIP_x02, SW3 SW_SPST, U1 AP2112K-3.3, U2 XIAO-ESP32-S3-DIP, U3 74AHCT1G125, U4 SN65HVD230

Commit message: Add DriverDasyChain schematic backup from September 8, 2026
Parts:
- removed C13: 4.7n, Capacitor_SMD:C_0603_1608Metric_Pad1.08x0.95mm_HandSolder, symbol Device:C
- removed D3: SMAJ5.0CA, Diode_SMD:D_SMA, symbol Diode:SMAJ5.0CA
- removed F1: Polyfuse, Fuse:Fuse_Bourns_MF-RHT050, symbol Device:Polyfuse
- removed J10, J12: Conn_01x04, TerminalBlock_WAGO:TerminalBlock_WAGO_2601-3104_1x04_P3.50mm_Vertical, symbol Connector_Generic:Conn_01x04
- removed R12, R13: 60.4, Resistor_SMD:R_0603_1608Metric_Pad0.98x0.95mm_HandSolder, symbol Device:R
- removed SW1: SW_DIP_x02, Button_Switch_SMD:SW_DIP_SPSTx02_Slide_6.7x6.64mm_W6.73mm_P2.54mm_LowProfile_JPin, symbol Switch:SW_DIP_x02
- removed SW3: SW_SPST, Button_Switch_SMD:SW_DIP_SPSTx01_Slide_Copal_CHS-01A_W5.08mm_P1.27mm_JPin, symbol Switch:SW_SPST
- added D2: SMAJ5.0A, Diode_SMD:D_SMA, symbol Diode:SMAJ5.0A
- added J11, J9: Conn_01x07_Socket, symbol Connector:Conn_01x07_Socket
- added J12, J13: Conn_01x03, TerminalBlock_WAGO:TerminalBlock_WAGO_2601-3104_1x04_P3.50mm_Vertical, symbol Connector_Generic:Conn_01x03
- added J7, J8: Conn_01x07_Pin, Connector_PinHeader_2.54mm:PinHeader_1x07_P2.54mm_Vertical, symbol Connector:Conn_01x07_Pin
- added R5: 120, Resistor_SMD:R_0603_1608Metric_Pad0.98x0.95mm_HandSolder, symbol Device:R
- added SW2: SW_SPST, Button_Switch_SMD:SW_DIP_SPSTx01_Slide_Copal_CHS-01A_W5.08mm_P1.27mm_JPin, symbol Switch:SW_SPST
- added TH1: Thermistor_PTC, symbol Device:Thermistor_PTC
- C6: value 2.2u -> 1u
- R11: value 470 -> R
- R8: value 6.8k -> 10k
Connections:
- net BRAKE +48V is gone; now on net +48V: J3.1 (Pin_1)
- net +3.3V: now also J7.3 (Pin_3)
- net +48V: now also J12.2 (Pin_2), J13.2 (Pin_2)
- net +5V: now also J5.1 (Pin_1), D2.1 (A1), J12.3 (Pin_3), J13.3 (Pin_3); no longer J5.3 (Pin_3)
- net CAN RX: now also J7.5 (Pin_5); no longer U2.10 (GPIO8_A9_D9_MISO)
- net CAN TX: now also J7.4 (Pin_4); no longer U2.11 (GPIO9_A10_D10_MOSI)
- net CANH: now also R5.2
- net CANL: now also SW2.1 (A)
- net GND: now also D2.2 (A2), J12.1 (Pin_1), J13.1 (Pin_1), J7.2 (Pin_2); no longer U2.13 (GND)
- net GPIO D0 (XIAO-ESP32-S3): now also J8.7 (Pin_7); no longer U2.1 (GPIO1_A0_D0)
- net GPIO D1 (XIAO-ESP32-S3): now also J8.6 (Pin_6); no longer U2.2 (GPIO2_A1_D1)
- net GPIO D3 (XIAO-ESP32-S3): now also J8.4 (Pin_4); no longer U2.4 (GPIO4_A3_D3)
- net GPIO D6 (XIAO-ESP32-S3): now also J8.1 (Pin_1); no longer U2.7 (GPIO43_D6_TX)
- net GPIO D7 (XIAO-ESP32-S3): now also J7.7 (Pin_7); no longer U2.8 (GPIO44_D7_RX)
- net at U2.12 (3V3): now also J9.3 (Pin_3)
- net at U2.14 (VBUS): now also J9.1 (Pin_1)
- net at U2.5 (GPIO5_A4_D4_SDA): now also J11.3 (Pin_3)
- net at U2.6 (GPIO6_A5_D5_SCL): now also J11.2 (Pin_2)
- net at U2.9 (GPIO7_A8_D8_SCK): now also J9.6 (Pin_6)
- net BRAKE GATE: no longer names the net of Q2.1 (G), R2.2, R4.1
- net BRAKE GATE: now also C10.1, J5.3 (Pin_3), R1.1, R9.2
- net BRAKE Out renamed MOSFET Out
- net MOSFET Out: now also TH1.2; no longer J3.2 (Pin_2)
- net Driver Out renamed Treiber Out
- net GPIO D2 (XIAO-ESP32-S3): no longer names the net of U2.3 (GPIO3_A2_D2)
- net GPIO D2 (XIAO-ESP32-S3): now also J11.5 (Pin_5); no longer R11.1
- removed net TLE4905L Out: C10.1, J5.1 (Pin_1), R1.1, R9.2
- new net: J11.7 (Pin_7), U2.1 (GPIO1_A0_D0)
- new net: J9.5 (Pin_5), U2.10 (GPIO8_A9_D9_MISO)
- new net: J9.4 (Pin_4), U2.11 (GPIO9_A10_D10_MOSI)
- new net: J9.2 (Pin_2), U2.13 (GND)
- new net: J11.6 (Pin_6), U2.2 (GPIO2_A1_D1)
- new net: J11.4 (Pin_4), U2.4 (GPIO4_A3_D3)
- new net: J11.1 (Pin_1), U2.7 (GPIO43_D6_TX)
- new net: J9.7 (Pin_7), U2.8 (GPIO44_D7_RX)
- new net: J3.2 (Pin_2), TH1.1
- new net: R5.1, SW2.2 (B)
- new net GPIO D5# (XIAO-ESP32-S3): J8.2 (Pin_2), R11.1
Other:
- moved on the sheet: C1, C10, C11, C12, C2, C3, C4, C5, C6, C7, C8, C9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
