File: PCB/KiCad/DriverDasyChain.kicad_sch (KiCad schematic)
At the start: 44 parts, among them J1 Conn_01x03, J10 Conn_01x04, J12 Conn_01x04, J2 Conn_01x03, J3 Conn_01x03, J4 Conn_01x04, J5 Conn_01x03, J6 Conn_01x04, Q2 Q_NMOS_GDS, SW1 SW_DIP_x02, SW3 SW_SPST, U1 AP2112K-3.3, U2 XIAO-ESP32-S3-DIP, U3 74AHCT1G125, U4 SN65HVD230

Commit message: Add Mouser order list for PCB components
- Created a new CSV file containing the order details for various components needed for the PCB assembly.
- Included manufacturer names, part numbers, quantities, designators, descriptions, and additional notes for each component.
Parts:
- removed SW3: SW_SPST, Button_Switch_SMD:SW_DIP_SPSTx01_Slide_Copal_CHS-01A_W5.08mm_P1.27mm_JPin, symbol Switch:SW_SPST
- added R14, R5: 220, Resistor_SMD:R_0603_1608Metric_Pad0.98x0.95mm_HandSolder, symbol Device:R
- added SW2: SW_SPDT, Button_Switch_SMD:SW_SPDT_PCM12, symbol Switch:SW_SPDT
Connections:
- net +3.3V: now also SW2.1 (A)
- net +5V: now also J5.1 (Pin_1); no longer J5.3 (Pin_3)
- net GPIO D6 (XIAO-ESP32-S3): now also R14.2; no longer J6.2 (Pin_2)
- net GPIO D7 (XIAO-ESP32-S3): now also R5.1; no longer J6.3 (Pin_3)
- net TLE4905L Out: now also J5.3 (Pin_3); no longer J5.1 (Pin_1)
- net at U2.12 (3V3): now also SW2.2 (B)
- new net: J6.2 (Pin_2), R14.1
- new net: J6.3 (Pin_3), R5.2
Other:
- note added: "UART Ausgang für möglich Debuging 220 Ohm um 5V Strom begrenze"
- note removed: "UART Ausgang für möglich Debuging"
- moved on the sheet: J5, J6

Commit message: Refactor PCB files and update documentation
- Deleted lock file for the PCB layout.
- Updated lock file for the schematic with new hostname.
- Modified PCB daisy chain documentation to clarify connections and component specifications, including:
  - Revised homing sensor pinout.
  - Added new component for CAN-TVS protection.
  - Adjusted capacitor counts and specifications.
  - Updated notes regarding BOM and assembly instructions.
- Created a new design rule file to enforce solid zone connections for power terminals on specific footprints.
Parts:
- removed C2, C3: 100u, Capacitor_THT:CP_Radial_D10.0mm_P5.00mm, symbol Device:C
- removed D1: US2DA, Diode_SMD:D_SMA, symbol Diode:US2DA
- added C14, C2, C3: 100u, Capacitor_THT:CP_Radial_D10.0mm_P5.00mm, symbol Device:C_Polarized
- added D1: US1D, Diode_SMD:D_SMA, symbol Diode:US1D
- added D2: PESD12VL2BT, Package_TO_SOT_SMD:SOT-23, symbol Power_Protection:NUP2105L
- added H1, H2, H3, H4: MountingHole, MountingHole:MountingHole_2.2mm_M2_Pad_TopBottom, symbol Mechanical:MountingHole
- F1: value Polyfuse -> 60R050XU; footprint Fuse:Fuse_Bourns_MF-RHT050 -> R0192:Fuse_Littelfuse_60R050XU
- J6: Note nur Platzhalter -> nicht auflöten -> (none)
- Q2: value Q_NMOS_GDS -> IRLR3410TRPBF
Connections:
- net +48V: now also C14.1, C2.1, C3.1, D1.1 (K)
- net BRAKE Out: now also D1.2 (A)
- net CANH: now also D2.1 (K)
- net CANL: now also D2.2 (K)
- net GND: now also C14.2, C2.2, C3.2, D2.3 (A)
- no-connect marks 6 -> 7
Other:
- note added: "Mouting Holes"
- moved on the sheet: C1, C10, C11, C12, C13, C4, C5, C6, C7, C8, C9, D3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
